File: Board.sch (EAGLE design)
At the start: 147 parts, among them U2 MAX7219CWG, U3 MAX7219CWG

Commit message: fixed wrong footprint for MAX7219
Parts:
- U2, U3: device maxim:MAX7219CWG -> max7219:MAX7219CWG
Changed lines of the file:
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@@
 </classes>
 <parts>
-<part name="U2" library="maxim" deviceset="MAX7219CWG" device=""/>
+<part name="U2" library="max7219" deviceset="MAX7219CWG" device=""/>
 <part name="LED1" library="led" deviceset="LED" device="CHIPLED_0805"/>
 <part name="LED2" library="led" deviceset="LED" device="CHIPLED_0805"/>
@@
 <part name="LED63" library="led" deviceset="LED" device="CHIPLED_0805"/>
 <part name="LED64" library="led" deviceset="LED" device="CHIPLED_0805"/>
-<part name="U3" library="maxim" deviceset="MAX7219CWG" device=""/>
+<part name="U3" library="max7219" deviceset="MAX7219CWG" device=""/>
 <part name="LED65" library="led" deviceset="LED" device="CHIPLED_0805"/>
 <part name="LED66" library="led" deviceset="LED" device="CHIPLED_0805"/>
